Commit message: Init + px4

File: urdf/seabed.xacro (robot description, xacro)
@@ -9,5 +9,5 @@
     <visual>
       <geometry>
-        <mesh filename="file://$(find floatgen)/meshes/$(arg seabed).ive"
+        <mesh filename="file://$(find drone_sim_environment)/meshes/$(arg seabed).ive"
               scale="${scale} ${scale} 1"/>
       </geometry>

File: urdf/turbine.xacro (robot description, xacro)
@@ -48,5 +48,5 @@
       <visual>
         <geometry>
-          <mesh filename="package://floatgen/meshes/pole.dae" scale="1 1 1"/>
+          <mesh filename="package://drone_sim_environment/meshes/pole.dae" scale="1 1 1"/>
         </geometry>
       </visual>
@@ -62,5 +62,5 @@
       <visual>
         <geometry>
-          <mesh filename="package://floatgen/meshes/blades.dae" scale="1 1 1"/>
+          <mesh filename="package://drone_sim_environment/meshes/blades.dae" scale="1 1 1"/>
         </geometry>
       </visual>
